File: KinesisMod/kicad_port.kicad_pcb (KiCad board)
At the start: 2 copper layers, 100 x 86 mm, 19 parts, among them J1 Conn_01x13, J2 Conn_01x13, J3 Conn_01x13, J4 Conn_01x13, J5 Conn_01x10, J6 Conn_01x10, M1 MountingHole_6.4mm_M6, M2 MountingHole_4.3mm_M4, M3 MountingHole_4.3mm_M4, M4 MountingHole_4.3mm_M4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

Commit message: Modify to support Teensy 4.x
Parts:
- removed M2: MountingHole_4.3mm_M4, Mounting_Holes:MountingHole_4.3mm_M4
- added H1: mounting pad, MountingHole:MountingHole_4.3mm_M4_Pad, F.Cu at (150.0, 106.0)
- U1: value Teensy++_2_0 -> Teensy4.1; footprint teensy:Teensy++_2_0_40p -> teensy:Teensy41
- moved U1 4.50 mm to (145.5, 90.4), turned to 180 degrees
Connections:
- D1 pad 2: +5V -> /3V3
- D2 pad 2: +5V -> /3V3
- D3 pad 2: +5V -> /3V3
- D4 pad 2: +5V -> /3V3
- J1 pad 1: /PC5 -> /ROW_F1
- J1 pad 10: /PC6 -> /ROW_F2
- J1 pad 11: /PC5 -> /ROW_F1
- J1 pad 12: Net-(J1-Pad12) -> unconnected-(J1-Pad12)
- J1 pad 13: Net-(J1-Pad13) -> unconnected-(J1-Pad13)
- J1 pad 2: /PC6 -> /ROW_F2
- J1 pad 3: /PB5 -> /COL_5
- J1 pad 4: /PB5 -> /COL_5
- J1 pad 5: /PC4 -> /ROW_ESC
- J1 pad 6: /PB3 -> /COL_3
- J1 pad 7: /PC6 -> /ROW_F2
- J1 pad 8: /PC5 -> /ROW_F1
- J1 pad 9: /PB4 -> /COL_4
- J2 pad 1: Net-(J2-Pad1) -> unconnected-(J2-Pad1)
- J2 pad 10: /PC6 -> /ROW_F2
- J2 pad 11: /PC5 -> /ROW_F1
- J2 pad 12: /PC4 -> /ROW_ESC
- J2 pad 13: /PB0 -> /COL_0
- J2 pad 2: Net-(J2-Pad2) -> unconnected-(J2-Pad2)
- J2 pad 3: /PC6 -> /ROW_F2
- J2 pad 4: /PC5 -> /ROW_F1
- J2 pad 5: Net-(J2-Pad5) -> unconnected-(J2-Pad5)
- J2 pad 6: /PB1 -> /COL_1
- J2 pad 7: /PC6 -> /ROW_F2
- J2 pad 8: /PC5 -> /ROW_F1
- J2 pad 9: /PB2 -> /COL_2
- J3 pad 1: /PC2 -> /ROW_0
- J3 pad 10: /PB4 -> /COL_4
- J3 pad 11: /PD7 -> /ROW_7
- J3 pad 12: /PC0 -> /ROW_8
- J3 pad 13: /PD6 -> /ROW_6
- J3 pad 2: /PC1 -> /ROW_9
- J3 pad 3: Net-(J3-Pad3) -> unconnected-(J3-Pad3)
- J3 pad 4: /PB0 -> /COL_0
- J3 pad 5: /PB1 -> /COL_1
- J3 pad 6: /PB2 -> /COL_2
- J3 pad 7: /PB3 -> /COL_3
- J3 pad 8: /PC3 -> /ROW_MIN
- J3 pad 9: Net-(J3-Pad9) -> unconnected-(J3-Pad9)
- J4 pad 1: /PB4 -> /COL_4
- J4 pad 10: /PD3 -> /ROW_3
- J4 pad 11: /PD4 -> /ROW_4
- J4 pad 12: /PD5 -> /ROW_5
- J4 pad 13: /PB0 -> /COL_0
- J4 pad 2: /PB3 -> /COL_3
- J4 pad 3: /PB2 -> /COL_2
- J4 pad 4: Net-(J4-Pad4) -> unconnected-(J4-Pad4)
- J4 pad 5: /PB1 -> /COL_1
- J4 pad 6: /PD0 -> /ROW_EQL
- J4 pad 7: /PD1 -> /ROW_1
- J4 pad 8: /PD2 -> /ROW_2
- J4 pad 9: Net-(J4-Pad9) -> unconnected-(J4-Pad9)
- J5 pad 1: Net-(J5-Pad1) -> unconnected-(J5-Pad1)
- J5 pad 10: Net-(J5-Pad10) -> unconnected-(J5-Pad10)
- J5 pad 2: Net-(J5-Pad2) -> unconnected-(J5-Pad2)
- J5 pad 3: /PD6 -> /ROW_6
- J5 pad 4: /PD7 -> /ROW_7
- J5 pad 5: /PC0 -> /ROW_8
- J5 pad 6: /PC1 -> /ROW_9
- J5 pad 7: /PB6 -> /COL_6
- J5 pad 8: /PB5 -> /COL_5
- J5 pad 9: Net-(J5-Pad9) -> unconnected-(J5-Pad9)
- J6 pad 1: /PD4 -> /ROW_4
- J6 pad 10: Net-(J6-Pad10) -> unconnected-(J6-Pad10)
- J6 pad 2: /PD2 -> /ROW_2
- J6 pad 3: /PD5 -> /ROW_5
- J6 pad 4: /PB6 -> /COL_6
- J6 pad 5: /PB5 -> /COL_5
- J6 pad 6: Net-(J6-Pad6) -> unconnected-(J6-Pad6)
- J6 pad 7: Net-(J6-Pad7) -> unconnected-(J6-Pad7)
- J6 pad 8: /PD3 -> /ROW_3
- J6 pad 9: Net-(J6-Pad9) -> unconnected-(J6-Pad9)
- R1 pad 2: /PF3 -> /LED_CAPS_LOCK
- R2 pad 2: /PF2 -> /LED_NUM_LOCK
- R3 pad 2: /PF1 -> /LED_SCROLL_LOCK
- R4 pad 2: /PF0 -> /LED_KEYPAD
- U1 pad 10: /PD7 -> /ROW_EQL
- U1 pad 11: /PE0 -> /ROW_1
- U1 pad 12: /PE1 -> /ROW_2
- U1 pad 13: /PC0 -> /ROW_3
- U1 pad 14: /PC1 -> /LED_CAPS_LOCK
- U1 pad 15: /PC2 -> unconnected-(U1-Pad15)
- U1 pad 16: /PC3 -> /LED_KEYPAD
- U1 pad 17: /PC4 -> /LED_SCROLL_LOCK
- U1 pad 18: /PC5 -> /LED_NUM_LOCK
- U1 pad 19: /PC6 -> unconnected-(U1-Pad19)
- U1 pad 2: /PB7 -> /ROW_0
- U1 pad 20: /PC7 -> unconnected-(U1-Pad20)
- U1 pad 21: +5V -> unconnected-(U1-Pad21)
- U1 pad 22: /PB6 -> unconnected-(U1-Pad22)
- U1 pad 23: /PB5 -> unconnected-(U1-Pad23)
- U1 pad 24: /PB4 -> unconnected-(U1-Pad24)
- U1 pad 25: /PB3 -> unconnected-(U1-Pad25)
- U1 pad 26: /PB2 -> unconnected-(U1-Pad26)
- U1 pad 27: /PB1 -> unconnected-(U1-Pad27)
- U1 pad 28: /PB0 -> unconnected-(U1-Pad28)
- U1 pad 29: /PE7 -> unconnected-(U1-Pad29)
- U1 pad 3: /PD0 -> /ROW_9
- U1 pad 30: /PE6 -> unconnected-(U1-Pad30)
- U1 pad 31: GND -> unconnected-(U1-Pad31)
- U1 pad 32: Net-(U1-Pad32) -> unconnected-(U1-Pad32)
- U1 pad 33: /PF0 -> unconnected-(U1-Pad33)
- U1 pad 34: /PF1 -> unconnected-(U1-Pad34)
- U1 pad 35: /PF2 -> unconnected-(U1-Pad35)
- U1 pad 36: /PF3 -> /COL_1
- U1 pad 37: /PF4 -> /COL_2
- U1 pad 38: /PF5 -> /ROW_5
- U1 pad 39: /PF6 -> /ROW_ESC
- U1 pad 4: /PD1 -> /ROW_MIN
- U1 pad 40: /PF7 -> /COL_0
- U1 pad 5: /PD2 -> /ROW_7
- U1 pad 6: /PD3 -> /ROW_8
- U1 pad 7: /PD4 -> /ROW_6
- U1 pad 8: /PD5 -> /COL_6
- U1 pad 9: /PD6 -> /ROW_4
Routing:
- net /COL_5: track 0.00 -> 215.2 mm, vias 0 -> 1
- net /COL_2: track 0.00 -> 203.1 mm, vias 0 -> 1
- net /COL_1: track 0.00 -> 196.3 mm, vias 0 -> 2
- net /PB5: track 196.1 -> 0.00 mm
- net /COL_3: track 0.00 -> 191.6 mm, vias 0 -> 2
- net /COL_4: track 0.00 -> 186.7 mm, vias 0 -> 2
- net /COL_0: track 0.00 -> 183.5 mm, vias 0 -> 1
- net /PB1: track 173.0 -> 0.00 mm
- net /PB2: track 163.3 -> 0.00 mm
- net /PB3: track 161.4 -> 0.00 mm
- net /PB4: track 159.4 -> 0.00 mm
- net /ROW_F1: track 0.00 -> 153.0 mm, vias 0 -> 2
- net /COL_6: track 0.00 -> 149.9 mm, vias 0 -> 1
- net /PB0: track 149.8 -> 0.00 mm
- net /ROW_ESC: track 0.00 -> 149.0 mm, vias 0 -> 1
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- added copper zone on B.Cu, net GND
- added copper zone on F.Cu, net GND
Other:
- net class Default removed
- rule pad_to_mask_clearance: 0.2 -> 0
- board text added: "Kinesis Contoured/Advantage Teensy 4.x + QMK Mod Fork of gitlab.com/Silman/kinesismod by dcpedit"
- board text removed: "Kinesis Contoured/Advantage Teensy++ 2.0 QMK Firmware Mod V1.0 RevA Redesign by Aaron Silman 2019-02 Based on work by Michael Stapelberg"
