File: blackpill/kicad_port.kicad_sch (KiCad schematic)
At the start: 16 parts, among them J1 Conn_01x13, J2 Conn_01x13, J3 Conn_01x13, J4 Conn_01x13, J5 Conn_01x10, J6 Conn_01x10, U1 YAAJ_WeAct_BlackPill_Part_Lik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

Commit message: Add Advantage compatibility
Parts:
- added D5: D_Small, symbol Device:D_Small
- added SW1: RotaryEncoder_Switch, symbol Device:RotaryEncoder_Switch
Connections:
- net COL_4: now also SW1.S2
- net GND: now also SW1.C
- net ROW_0: now also D5.1 (K)
- net ENB: now reaches U1.42 (SWCLK)
- net ENB: now also SW1.B
- net ENA: now reaches U1.43 (SWIO)
- net ENA: now also SW1.A
- new net: D5.2 (A), SW1.S1
- no-connect marks 31 -> 29
Changed lines of the file:
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@@
   (no_connect (at 156.21 36.83))
   (no_connect (at 67.31 93.98))
-  (no_connect (at 133.35 82.55))
-  (no_connect (at 130.81 82.55))
   (no_connect (at 191.77 139.7))
   (no_connect (at 71.12 140.97))
@@
     (stroke (width 0) (type default) (color 0 0 0 0))
   )
+  (wire (pts (xy 139.7 105.41) (xy 144.78 105.41))
+    (stroke (width 0) (type default) (color 0 0 0 0))
+  )
   (wire (pts (xy 67.31 96.52) (xy 69.85 96.52))
     (stroke (width 0) (type default) (color 0 0 0 0))
@@
     (stroke (width 0) (type default) (color 0 0 0 0))
   )
+  (wire (pts (xy 124.46 110.49) (xy 114.3 110.49))
+    (stroke (width 0) (type default) (color 0 0 0 0))
+  )
   (wire (pts (xy 67.31 45.72) (xy 69.85 45.72))
     (stroke (width 0) (type default) (color 0 0 0 0))
@@
     (stroke (width 0) (type default) (color 0 0 0 0))
   )
+  (wire (pts (xy 133.35 82.55) (xy 133.35 92.71))
+    (stroke (width 0) (type default) (color 0 0 0 0))
+  )
+  (wire (pts (xy 149.86 105.41) (xy 160.02 105.41))
+    (stroke (width 0) (type default) (color 0 0 0 0))
+  )
   (wire (pts (xy 67.31 38.1) (xy 69.85 38.1))
     (stroke (width 0) (type default) (color 0 0 0 0))
@@
     (stroke (width 0) (type default) (color 0 0 0 0))
   )
+  (wire (pts (xy 139.7 110.49) (xy 149.86 110.49))
+    (stroke (width 0) (type default) (color 0 0 0 0))
+  )
   (wire (pts (xy 146.05 152.4) (xy 146.05 149.86))
     (stroke (width 0) (type default) (color 0 0 0 0))
@@
     (stroke (width 0) (type default) (color 0 0 0 0))
   )
+  (wire (pts (xy 130.81 82.55) (xy 130.81 92.71))
+    (stroke (width 0) (type default) (color 0 0 0 0))
+  )
   (wire (pts (xy 67.31 71.12) (xy 69.85 71.12))
     (stroke (width 0) (type default) (color 0 0 0 0))
@@
     (stroke (width 0) (type default) (color 0 0 0 0))
   )
+  (wire (pts (xy 124.46 105.41) (xy 114.3 105.41))
+    (stroke (width 0) (type default) (color 0 0 0 0))
+  )
   (wire (pts (xy 179.07 139.7) (xy 179.07 137.16))
     (stroke (width 0) (type default) (color 0 0 0 0))
@@
     (effects (font (size 1.27 1.27)) (justify left bottom))
   )
+  (label "COL_4" (at 149.86 110.49 180)
+    (effects (font (size 1.27 1.27)) (justify right bottom))
+  )
   (label "ROW_1" (at 93.98 59.69 0)
     (effects (font (size 1.27 1.27)) (justify left bottom))
@@
     (effects (font (size 1.27 1.27)) (justify left bottom))
   )
+  (label "ENA" (at 114.3 105.41 0)
+    (effects (font (size 1.27 1.27)) (justify left bottom))
+  )
   (label "ROW_MIN" (at 93.98 31.75 0)
     (effects (font (size 1.27 1.27)) (justify left bottom))
@@
     (effects (font (size 1.27 1.27)) (justify right bottom))
   )
+  (label "ROW_0" (at 160.02 105.41 180)
+    (effects (font (size 1.27 1.27)) (justify right bottom))
+  )
   (label "ROW_8" (at 181.61 137.16 90)
     (effects (font (size 1.27 1.27)) (justify left bottom))
@@
     (effects (font (size 1.27 1.27)) (justify left bottom))
   )
+  (label "ENA" (at 130.81 92.71 90)
+    (effects (font (size 1.27 1.27)) (justify left bottom))
+  )
   (label "LED_SCROLL_LOCK" (at 133.35 152.4 270)
     (effects (font (size 1.27 1.27)) (justify right bottom))
@@
     (effects (font (size 1.27 1.27)) (justify left bottom))
   )
+  (label "ENB" (at 133.35 92.71 90)
+    (effects (font (size 1.27 1.27)) (justify left bottom))
+  )
   (label "COL_2" (at 69.85 96.52 0)
     (effects (font (size 1.27 1.27)) (justify left bottom))
@@
   )
   (label "ROW_5" (at 86.36 138.43 90)
+    (effects (font (size 1.27 1.27)) (justify left bottom))
+  )
+  (label "ENB" (at 114.3 110.49 0)
     (effects (font (size 1.27 1.27)) (justify left bottom))
   )
@@
     (pin "1")
   )
+  (symbol (lib_id "Device:D_Small") (at 147.32 105.41 0) (mirror y) (unit 1)
+    (in_bom yes) (on_board yes) (fields_autoplaced)
+    (property "Reference" "D5" (id 0) (at 147.32 100.4275 0))
+    (property "Value" "D_Small" (id 1) (at 147.32 103.2026 0))
+    (property "Footprint" "" (id 2) (at 147.32 105.41 90)
+      (effects (font (size 1.27 1.27)) hide)
+    )
+    (property "Datasheet" "~" (id 3) (at 147.32 105.41 90)
+      (effects (font (size 1.27 1.27)) hide)
+    )
+    (pin "1")
+    (pin "2")
+  )
   (symbol (lib_id "Mechanical:MountingHole_Pad") (at 87.63 116.84 270) (unit 1)
     (in_bom yes) (on_board yes)
@@
     (pin "1")
   )
+  (symbol (lib_id "kicad_port-rescue:GND-power") (at 124.46 107.95 270) (mirror x) (unit 1)
+    (in_bom yes) (on_board yes)
+    (property "Reference" "#PWR0103" (id 0) (at 118.11 107.95 0)
+      (effects (font (size 1.27 1.27)) hide)
+    )
+    (property "Value" "GND" (id 1) (at 121.2088 107.823 90)
+      (effects (font (size 1.27 1.27)) (justify right))
+    )
+    (property "Footprint" "" (id 2) (at 124.46 107.95 0)
+      (effects (font (size 1.27 1.27)) hide)
+    )
+    (property "Datasheet" "" (id 3) (at 124.46 107.95 0)
+      (effects (font (size 1.27 1.27)) hide)
+    )
+    (pin "1")
+  )
   (symbol (lib_id "kicad_port-rescue:GND-power") (at 156.21 29.21 90) (unit 1)
     (in_bom yes) (on_board yes)
@@
     )
     (pin "1")
+  )
+  (symbol (lib_id "Device:RotaryEncoder_Switch") (at 132.08 107.95 0) (unit 1)
+    (in_bom yes) (on_board yes) (fields_autoplaced)
+    (property "Reference" "SW1" (id 0) (at 132.08 98.9035 0))
+    (property "Value" "RotaryEncoder_Switch" (id 1) (at 132.08 101.6786 0))
+    (property "Footprint" "" (id 2) (at 128.27 103.886 0)
+      (effects (font (size 1.27 1.27)) hide)
+    )
+    (property "Datasheet" "~" (id 3) (at 132.08 101.346 0)
+      (effects (font (size 1.27 1.27)) hide)
+    )
+    (pin "A")
+    (pin "B")
+    (pin "C")
+    (pin "S1")
+    (pin "S2")
   )
   (symbol (lib_id "YAAJ_WeAct_BlackPill_Part_Like_SWD_Breakout:YAAJ_WeAct_BlackPill_Part_Like_SWD_Breakout") (at 133.35 49.53 0) (unit 1)
@@
       (reference "#PWR0102") (unit 1) (value "GND") (footprint "")
     )
+    (path "/4e47e4af-bbb8-4836-acf7-ed8caa23763c"
+      (reference "#PWR0103") (unit 1) (value "GND") (footprint "")
+    )
     (path "/00000000-0000-0000-0000-00005c6b70ab"
       (reference "#PWR0106") (unit 1) (value "GND") (footprint "")
@@
       (reference "D4") (unit 1) (value "LED_ALT") (footprint "LED_THT:LED_D3.0mm")
     )
+    (path "/1114fad5-081a-4442-a66d-0aef7480e33f"
+      (reference "D5") (unit 1) (value "D_Small") (footprint "")
+    )
     (path "/261e7774-9f95-4d32-8ff3-370c3bfbbb38"
       (reference "H1") (unit 1) (value "mounting pad") (footprint "MountingHole:MountingHole_4.3mm_M4_Pad")
@@
       (reference "R4") (unit 1) (value "R_US") (footprint "Resistor_THT:R_Axial_DIN0204_L3.6mm_D1.6mm_P5.08mm_Horizontal")
     )
+    (path "/a54a2d51-4b66-4d14-b33d-1444b55de06d"
+      (reference "SW1") (unit 1) (value "RotaryEncoder_Switch") (footprint "")
+    )
     (path "/c581271b-42f0-4e3f-b8c9-a824614bb7e7"

Commit message: Update readme with wireless info
Parts:
- added J7, J8: Conn_01x13, kinesisMod_board_connectors:Molex_0039532135, symbol kicad_port-rescue:Conn_01x13-Connector_Generic
Connections:
- net 3V3: now also U1.20 (3V3); no longer U1.44 (3V3)
- net COL_5: now also J7.8 (Pin_8), J8.9 (Pin_9)
- net COL_6: now also J7.7 (Pin_7), J8.10 (Pin_10)
- net ROW_2: now also J8.12 (Pin_12)
- net ROW_3: now also J8.6 (Pin_6)
- net ROW_4: now also J8.13 (Pin_13)
- net ROW_5: now also J8.11 (Pin_11)
- net ROW_6: now also J7.3 (Pin_3)
- net ROW_7: now also J7.4 (Pin_4)
- net ROW_8: now also J7.5 (Pin_5)
- net ROW_9: now also J7.6 (Pin_6)
- no-connect marks 29 -> 36
Other:
- moved on the sheet: J5, J6
